File: Fall-2026/embedded-systems/ESP32/ESP32.kicad_sch (KiCad schematic)
At the start: 0 parts

Commit message: finished lab 2 library
Parts:
- added D1, D2, D3: Red, symbol Wright_State_Library:LED_RED_0603
- added D4, D5: Yellow, RF_Module:ESP32-S3-WROOM-2, symbol Wright_State_Library:LED_YELLOW_0603
- added D6, D7, D8, D9: Green, symbol Wright_State_Library:LED_GREEN_0603
- added R1, R2, R3, R4, R5, R6, R7, R8: 330, ESP32_30pin, symbol Wright_State_Library:R330_1%_0603
- added R10, R9: 10K, symbol Wright_State_Library:R10K_1%_0603
- added R11: 1K, symbol Wright_State_Library:R1K_1%_0603
- added SW1, SW2: (no value), symbol Wright_State_Library:SWITCH_0603
- added TP1, TP2: (no value), symbol Wright_State_Library:TEST_POINT_0603
- added U1: (no value), ESP32_30pin, symbol Wright_State_Library:ESP32_30Pin
Connections:
- new net: D7.1, R7. (2)
- new net: TP1.1, U1.26 (GPIO21)
- new net: D4.1, R4. (2)
- new net: D9.1, R11. (2)
- new net: D2.1, R2. (2)
- new net: D6.1, R6. (2)
- new net: D5.1, R5. (2)
- new net: D3.1, R3. (2)
- new net: D8.1, R8. (2)
- new net: D1.1, R1. (2)
- new net +3.3V: R10. (2), R11. (2), R9. (2), U1.16 (3.3v)
- new net GND: D1.2, D2.2, D3.2, D4.2, D5.2, D6.2, D7.2, D8.2, D9.2, SW1.2, SW2.2, TP2.1
- new net LED1: R1. (2), U1.10 (GPIO32)
- new net LED2: R2. (2), U1.9 (GPIO33)
- new net LED3: R3. (2), U1.8 (GPIO25)
- new net LED4: R4. (2), U1.7 (GPIO26)
- new net LED5: R5. (2), U1.30 (GPIO23), U1.6 (GPIO27)
- new net LED6: R6. (2), U1.5 (GPIO14)
- new net LED7: R7. (2), U1.3 (GPIO13)
- new net LED8: R8. (2)
- new net NETSW1: R9. (2), SW1.1, U1.25 (GPIO19)
- new net NETSW2: R10. (2), SW2.1, U1.24 (GPIO18)
