File: Fall-2026/embedded-systems/ESP32/ESP32.kicad_sch (KiCad schematic)
At the start: 25 parts

Commit message: finished embedded systems lab 4
Parts:
- D1, D2, D3, D6, D7, D8, D9: footprint (none) -> LED_SMD:LED_0603_1608Metric_Pad1.05x0.95mm_HandSolder
- D4, D5: footprint RF_Module:ESP32-S3-WROOM-2 -> LED_SMD:LED_0603_1608Metric_Pad1.05x0.95mm_HandSolder
- R1, R2, R3, R4, R5, R6, R7, R8: footprint ESP32_30pin -> Resistor_SMD:R_0603_1608Metric
- R10, R11, R9: footprint (none) -> Resistor_SMD:R_0603_1608Metric
- SW1, SW2: footprint (none) -> WrightStateFootprint:TL2233
- TP1, TP2: footprint (none) -> TestPoint:TestPoint_Pad_D2.0mm
- U1: footprint ESP32_30pin -> WrightStateFootprint:ESP32_30pin
Connections:
- net +3.3V: now also R10.2, R11.1, R9.2; no longer R10. (2), R11. (2), R9. (2)
- net LED1: now also R1.1; no longer R1. (2)
- net LED2: now also R2.1; no longer R2. (2)
- net LED3: now also R3.1; no longer R3. (2)
- net LED4: now also R4.1; no longer R4. (2)
- net LED5: now also R5.1; no longer R5. (2), U1.30 (GPIO23)
- net LED6: now also R6.1; no longer R6. (2)
- net LED7: now also R7.1; no longer R7. (2)
- net LED8: now also R8.1, U1.30 (GPIO23); no longer R8. (2)
- net NETSW1: now also R9.1; no longer R9. (2)
- net NETSW2: now also R10.1; no longer R10. (2)
- net at D7.1: now also R7.2; no longer R7. (2)
- net at D4.1: now also R4.2; no longer R4. (2)
- net at D9.1: now also R11.2; no longer R11. (2)
- net at D2.1: now also R2.2; no longer R2. (2)
- net at D6.1: now also R6.2; no longer R6. (2)
- net at D5.1: now also R5.2; no longer R5. (2)
- net at D3.1: now also R3.2; no longer R3. (2)
- net at D8.1: now also R8.2; no longer R8. (2)
- net at D1.1: now also R1.2; no longer R1. (2)
Other:
- moved on the sheet: U1

Commit message: working on traces for pcb lab
Connections:
- net GND: now also U1.17 (GND), U1.2 (GND)
- no-connect marks 18 -> 16
Changed lines of the file:
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@@
 	)
 	(no_connect
-		(at 151.13 80.01)
-	)
-	(no_connect
 		(at 151.13 87.63)
 	)
@@
 		(at 179.07 102.87)
 	)
-	(no_connect
-		(at 179.07 80.01)
-	)
 	(wire
 		(pts
@@
 	(wire
 		(pts
+			(xy 179.07 80.01) (xy 180.34 80.01)
+		)
+		(stroke
+			(width 0)
+			(type default)
+		)
+	)
+	(wire
+		(pts
 			(xy 236.22 121.92) (xy 238.76 121.92)
 		)
@@
 	(wire
 		(pts
+			(xy 180.34 80.01) (xy 180.34 78.74)
+		)
+		(stroke
+			(width 0)
+			(type default)
+		)
+	)
+	(wire
+		(pts
 			(xy 124.46 91.44) (xy 127 91.44)
 		)
@@
 	(wire
 		(pts
+			(xy 148.59 80.01) (xy 151.13 80.01)
+		)
+		(stroke
+			(width 0)
+			(type default)
+		)
+	)
+	(wire
+		(pts
 			(xy 223.52 71.12) (xy 224.79 71.12)
 		)
@@
 	)
 	(symbol
+		(lib_id "power:GND")
+		(at 148.59 80.01 0)
+		(unit 1)
+		(body_style 1)
+		(exclude_from_sim no)
+		(in_bom yes)
+		(on_board yes)
+		(in_pos_files yes)
+		(dnp no)
+		(property "Reference" "#PWR09"
+			(at 148.59 86.36 0)
+			(hide yes)
+			(show_name no)
+			(do_not_autoplace no)
+			(effects
+				(font
+					(size 1.27 1.27)
+				)
+			)
+		)
+		(property "Value" "GND"
+			(at 147.574 83.566 0)
+			(show_name no)
+			(do_not_autoplace no)
+			(effects
+				(font
+					(size 1.27 1.27)
+				)
+			)
+		)
+		(property "Footprint" ""
+			(at 148.59 80.01 0)
+			(hide yes)
+			(show_name no)
+			(do_not_autoplace no)
+			(effects
+				(font
+					(size 1.27 1.27)
+				)
+			)
+		)
+		(property "Datasheet" ""
+			(at 148.59 80.01 0)
+			(hide yes)
+			(show_name no)
+			(do_not_autoplace no)
+			(effects
+				(font
+					(size 1.27 1.27)
+				)
+			)
+		)
+		(property "Description" "Power symbol creates a global label with name \"GND\" , ground"
+			(at 148.59 80.01 0)
+			(hide yes)
+			(show_name no)
+			(do_not_autoplace no)
+			(effects
+				(font
+					(size 1.27 1.27)
+				)
+			)
+		)
+		(pin "1"
+		)
+		(instances
+			(project "ESP32"
+				(path "/41e687bb-bb38-436f-b2ad-ca9f4eebe283"
+					(reference "#PWR09")
+					(unit 1)
+				)
+			)
+		)
+	)
+	(symbol
 		(lib_id "Wright_State_Library:R1K_1%_0603")
 		(at 121.92 91.44 0)
@@
 					(unit 1)
 				)
+			)
+		)
+	)
+	(symbol
+		(lib_id "power:GND")
+		(at 180.34 78.74 90)
+		(unit 1)
+		(body_style 1)
+		(exclude_from_sim no)
+		(in_bom yes)
+		(on_board yes)
+		(in_pos_files yes)
+		(dnp no)
+		(property "Reference" "#PWR03"
+			(at 186.69 78.74 0)
+			(hide yes)
+			(show_name no)
+			(do_not_autoplace no)
+			(effects
+				(font
+					(size 1.27 1.27)
+				)
+			)
+		)
+		(property "Value" "GND"
+			(at 183.134 78.74 90)
+			(show_name no)
+			(do_not_autoplace no)
+			(effects
+				(font
+					(size 1.27 1.27)
+				)
+				(justify right)
+			)
+		)
+		(property "Footprint" ""
+			(at 180.34 78.74 0)
+			(hide yes)
+			(show_name no)
+			(do_not_autoplace no)
+			(effects
+				(font
+					(size 1.27 1.27)
+				)
+			)
+		)
+		(property "Datasheet" ""
+			(at 180.34 78.74 0)
+			(hide yes)
+			(show_name no)
+			(do_not_autoplace no)
+			(effects
+				(font
+					(size 1.27 1.27)
+				)
+			)
+		)
+		(property "Description" "Power symbol creates a global label with name \"GND\" , ground"
+			(at 180.34 78.74 0)
+			(hide yes)
+			(show_name no)
+			(do_not_autoplace no)
+			(effects
+				(font
+					(size 1.27 1.27)
+				)
+			)
+		)
+		(pin "1"
+		)
+		(instances
+			(project "ESP32"
+				(path "/41e687bb-bb38-436f-b2ad-ca9f4eebe283"
+					(reference "#PWR03")
+					(unit 1)
+				)
