File: Fall-2026/embedded-systems/ESP32/ESP32.kicad_pcb (KiCad board)
At the start: 2 copper layers, 26 x 49 mm, 25 parts

Commit message: working on traces for pcb lab
Parts:
- added REF**: Fiducial_0.5mm_Mask1.5mm, Fiducial:Fiducial_0.5mm_Mask1.5mm, F.Cu at (142.0, 129.5)
- added REF**: Fiducial_0.5mm_Mask1.5mm, Fiducial:Fiducial_0.5mm_Mask1.5mm, F.Cu at (197.5, 73.0)
- added REF**: Fiducial_0.5mm_Mask1.5mm, Fiducial:Fiducial_0.5mm_Mask1.5mm, F.Cu at (197.5, 129.5)
- moved D8 69.4 mm to (142.5, 116.5), turned to 180 degrees
- moved D7 69.1 mm to (142.5, 113.0), turned to 180 degrees
- moved D6 68.8 mm to (142.5, 109.5), turned to 180 degrees
- moved D5 68.5 mm to (142.5, 106.0), turned to 180 degrees
- moved D4 68.3 mm to (142.5, 102.5), turned to 180 degrees
- moved D3 68.0 mm to (142.5, 99.0), turned to 180 degrees
- moved D2 67.8 mm to (142.5, 95.5), turned to 180 degrees
- moved D1 67.6 mm to (142.5, 92.0), turned to 180 degrees
- moved R8 65.6 mm to (148.0, 116.5), turned to 180 degrees
- moved R7 65.3 mm to (148.0, 112.5), turned to 180 degrees
- moved R1 60.2 mm to (148.0, 93.0), turned to 180 degrees
- moved R2 60.2 mm to (148.0, 96.0), turned to 180 degrees
- moved R3 60.1 mm to (148.0, 99.0), turned to 180 degrees
- moved R4 60.1 mm to (148.0, 102.0), turned to 180 degrees
- moved R5 60.1 mm to (148.0, 105.0), turned to 180 degrees
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Connections:
- U1 pad 17: unconnected-(U1-GND-Pad17) -> GND
- U1 pad 2: unconnected-(U1-GND-Pad2) -> GND
Routing:
- net GND: track 0.00 -> 114.2 mm, vias 0 -> 2
- net /LED8: track 0.00 -> 54.5 mm, vias 0 -> 2
- net +3.3V: track 0.00 -> 30.5 mm, vias 0 -> 3
- net Net-(U1-GPIO21): track 0.00 -> 19.3 mm
- net /NETSW1: track 0.00 -> 12.7 mm
- net /NETSW2: track 0.00 -> 12.3 mm
- net Net-(D9-Pad1): track 0.00 -> 7.59 mm
- net /LED1: track 0.00 -> 5.68 mm
- net /LED2: track 0.00 -> 5.49 mm
- net /LED6: track 0.00 -> 5.33 mm
- net /LED3: track 0.00 -> 5.30 mm
- net /LED4: track 0.00 -> 5.11 mm
- net /LED7: track 0.00 -> 4.97 mm
- net /LED5: track 0.00 -> 4.93 mm
- net Net-(D6-Pad1): track 0.00 -> 4.21 mm
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- added copper zone on B.Cu, net +3.3V
- added copper zone on F.Cu, net GND
Other:
- rule pad_to_mask_clearance: 0 -> 0.0762

Commit message: finished pcb labs
Parts:
- moved TPGND1 58.4 mm to (150.0, 127.0)
- moved R11 4.78 mm to (189.7, 118.5), turned to 0 degrees
- moved R9 3.54 mm to (188.5, 93.3)
- moved D1 2.00 mm to (144.5, 92.0)
- moved D2 2.00 mm to (144.5, 95.5)
- moved D3 2.00 mm to (144.5, 99.0)
- moved D4 2.00 mm to (144.5, 102.5)
- moved D5 2.00 mm to (144.5, 106.0)
- moved D6 2.00 mm to (144.5, 109.5)
- moved D7 2.00 mm to (144.5, 113.0)
- moved D8 2.00 mm to (144.5, 116.5)
- moved D9 2.00 mm to (195.1, 117.5)
- moved R1 2.00 mm to (150.0, 93.0)
- moved R10 2.00 mm to (188.5, 99.3), turned to -90 degrees
- moved R2 2.00 mm to (150.0, 96.0)
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- renumbered TP2 to TPGND1, TP1 to TPSCOPE1
Routing:
- net GND: track 114.2 -> 38.4 mm, vias 2 -> 0
- net +3.3V: track 30.5 -> 4.05 mm
- net Net-(D9-Pad1): track 7.59 -> 4.16 mm
- net /LED8: track 54.5 -> 57.0 mm, vias 2 -> 0
Other:
- board size 26 x 49 mm -> 63.5 x 63.5 mm
